File: pcb-module/kunai-mod.kicad_sch (KiCad schematic)
At the start: 24 parts, among them J1 Outline, J2 SWD, Q1 UM6K33NTN, U1 NCP115AMX330TCG, U2 W25Q16JWXHIQ TR, U3 RP2040, Y1 ABM8-272-T3

Commit message: Add footprint and update readme, small tweaks to pcb/schematic.
Other:
- title: (none) -> Kunai module
Changed lines of the file:
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@@
 	(generator_version "9.0")
 	(paper "A")
+	(title_block
+		(title "Kunai module")
+		(date "2025-10-24")
+		(rev "0")
+	)
 	(junction
 		(at 132.08 43.18)
